File: PCB-DESIGN/devboard.kicad_sch (KiCad schematic)
At the start: 44 parts, among them J1 USB_C_Receptacle_USB2.0_14P, J2 Conn_01x20, J3 Conn_01x20, J4 Conn_01x03, SW1 SW_Push, U1 RP2040, U2 MCP1700x-330xxTT, U3 W25Q16JVUXIQ TR, U4 TMP112xxDRL, Y1 12 MHz

Commit message: Add files via upload
Parts:
- removed C20, C21: 0.1uF, Capacitor_SMD:C_0402_1005Metric, symbol Device:C
- removed D1: LED, LED_SMD:LED_0402_1005Metric, symbol Device:LED
- C1, C10, C11, C12, C15, C16, C17, C2, C3, C4, C5, C6, C7, C8, C9: footprint Capacitor_SMD:C_0402_1005Metric -> Capacitor_SMD:C_0603_1608Metric
- C13, C14: footprint Capacitor_SMD:C_0603_1608Metric -> Capacitor_SMD:C_0805_2012Metric
- C18, C19: value 0.1uF -> 10uF; footprint Capacitor_SMD:C_0402_1005Metric -> Capacitor_SMD:C_0603_1608Metric
- R1, R10, R11, R2, R3, R4, R5, R6, R7, R8, R9: footprint Resistor_SMD:R_0402_1005Metric -> Resistor_SMD:R_0603_1608Metric
Connections:
- net +3V3: now also C18.1, C19.1, D2.4 (VDD)
- net GND: now also C18.2, D2.2 (VSS), U4.2 (GND)
- net at SW1.2: now also R6.1
- net at R8.1: now also U4.5 (V+); no longer C18.1
Other:
- moved on the sheet: C18, R8, SW1
